File: krabi-actuator-board-v2.kicad_sch (KiCad schematic)
At the start: 27 parts, among them J1 Power, J2 PWM, J3 Analog, J4 PWM, J5 Analog, J6 Communication, J7 Digital, J8 Conn_01x02_Pin, U1 XGZP6897D_differential_pressu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, U2 XGZP6897D_differential_pressu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

Commit message: Assigning footprints to schemas
Parts:
- C1: footprint Capacitor_THT:CP_Radial_D5.0mm_P2.00mm -> Capacitor_THT:CP_Radial_D16.0mm_P7.50mm
- F1: footprint Resistor_THT:R_Axial_DIN0411_L9.9mm_D3.6mm_P15.24mm_Horizontal -> Inductor_SMD:L_Bourns-SRN1060
Changed lines of the file:
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@@
       (effects (font (size 1.27 1.27)))
     )
-    (property "Footprint" "Resistor_THT:R_Axial_DIN0411_L9.9mm_D3.6mm_P15.24mm_Horizontal" (at 35.56 182.118 90)
+    (property "Footprint" "Inductor_SMD:L_Bourns-SRN1060" (at 35.56 182.118 90)
       (effects (font (size 1.27 1.27)) hide)
     )
@@
       (effects (font (size 1.27 1.27)) (justify left))
     )
-    (property "Footprint" "Capacitor_THT:CP_Radial_D5.0mm_P2.00mm" (at 59.3852 187.96 0)
-      (effects (font (size 1.27 1.27)) hide)
-    )
+    (property "Footprint" "Capacitor_THT:CP_Radial_D16.0mm_P7.50mm" (at 59.3852 187.96 0)
+      (effects (font (size 1.27 1.27)) hide)
+    )

Commit message: Fixing bad association and symbols*
Parts:
- F1: footprint Inductor_SMD:L_Bourns-SRN1060 -> Resistor_THT:R_Axial_DIN0411_L9.9mm_D3.6mm_P15.24mm_Horizontal
Changed lines of the file:
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@@
     )
   )
-  (symbol (lib_id "power:GND") (at 43.18 45.72 0) (unit 1)
+  (symbol (lib_name "GND_2") (lib_id "power:GND") (at 43.18 45.72 0) (unit 1)
     (in_bom yes) (on_board yes) (dnp no)
     (property "Reference" "#PWR04" (at 43.18 52.07 0)
@@
     )
   )
-  (symbol (lib_id "power:GND") (at 76.2 45.72 0) (unit 1)
+  (symbol (lib_name "GND_1") (lib_id "power:GND") (at 76.2 45.72 0) (unit 1)
     (in_bom yes) (on_board yes) (dnp no)
     (property "Reference" "#PWR05" (at 76.2 52.07 0)
@@
     )
   )
-  (symbol (lib_id "power:+5V") (at 77.47 125.73 0) (unit 1)
+  (symbol (lib_name "+5V_1") (lib_id "power:+5V") (at 77.47 125.73 0) (unit 1)
     (in_bom yes) (on_board yes) (dnp no)
     (property "Reference" "#PWR06" (at 77.47 129.54 0)
@@
       (effects (font (size 1.27 1.27)))
     )
-    (property "Footprint" "Inductor_SMD:L_Bourns-SRN1060" (at 35.56 182.118 90)
-      (effects (font (size 1.27 1.27)) hide)
-    )
+    (property "Footprint" "Resistor_THT:R_Axial_DIN0411_L9.9mm_D3.6mm_P15.24mm_Horizontal" (at 35.56 182.118 90)
+      (effects (font (size 1.27 1.27)) hide)
+    )
