File: servos.kicad_sch (KiCad schematic)
At the start: 24 parts, among them J10 Conn_01x03_Male, J18 Conn_01x03_Male, J19 Conn_01x03_Male, J5 Conn_01x03_Male, J6 Conn_01x03_Male, J7 Conn_01x03_Male, J8 Conn_01x03_Male, J9 Conn_01x03_Male, Q5 DMN2011UTS, Q6 DMN2011UTS

Commit message: add DCDC 6V
Parts:
- removed D2, D3: D_Zener, Diode_SMD:D_1206_3216Metric, symbol Device:D_Zener
- removed D4: D, Diode_SMD:D_1206_3216Metric, symbol Device:D
- removed PS1, PS2: LM2596s module, LibraryVictor:lm2596Module, symbol New_Library_Victor:LM2596s module
- removed Q5: DMN2011UTS, Package_SO:TSSOP-8_4.4x3mm_P0.65mm, symbol New_Library_Victor:DMN2011UTS
- removed R1: 220R, Resistor_SMD:R_0603_1608Metric, symbol Device:R
Connections:
- net GND_POWER is gone; now on net GND: D5.2 (A), Q6.1 (S), Q6.2 (S), Q6.3 (S)
- net GND_SERVO_1 is gone; now on net GND_SERVO_2: D35.2 (A), J18.1 (Pin_1), J5.1 (Pin_1), J6.1 (Pin_1), J7.1 (Pin_1)

Commit message: fix warnings + separate enable for Steppers
Connections:
- net ENABLE_SERVO_POWER_2 renamed ENABLE_SERVO_POWER_1
Changed lines of the file:
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@@
 		)
 	)
-	(global_label "ENABLE_SERVO_POWER_2"
+	(global_label "ENABLE_SERVO_POWER_1"
 		(shape input)
 		(at 69.85 176.53 180)
@@
 		)
 		(property "Intersheetrefs" "${INTERSHEET_REFS}"
-			(at 43.7907 176.4506 0)
+			(at 43.2188 176.53 0)
 			(effects
 				(font

Commit message: change fuse + start servo order + routing
Connections:
- net SERVO_4: now also J18.3 (Pin_3); no longer J8.3 (Pin_3)
- net SERVO_5: now also J19.3 (Pin_3); no longer J9.3 (Pin_3)
- net SERVO_6: now also J8.3 (Pin_3); no longer J10.3 (Pin_3)
- net SERVO_7: now also J9.3 (Pin_3); no longer J18.3 (Pin_3)
- net SERVO_8: now also J10.3 (Pin_3); no longer J19.3 (Pin_3)
Changed lines of the file:
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@@
+		)
+	)
+	(global_label "SERVO_7"
+		(shape input)
+		(at 201.93 135.89 180)
+		(fields_autoplaced yes)
+		(effects
+			(font
+				(size 1.27 1.27)
+			)
+			(justify right)
+		)
+		(property "Intersheetrefs" "${INTERSHEET_REFS}"
+			(at 191.2921 135.8106 0)
+			(effects
+				(font
+					(size 1.27 1.27)
+				)
+				(justify right)
+				(hide yes)
+			)
+		)
+	)
+	(global_label "GND"
+		(shape input)
+		(at 129.54 72.39 180)
+		(fields_autoplaced yes)
+		(effects
+			(font
+				(size 1.27 1.27)
+			)
+			(justify right)
+		)
+		(property "Intersheetrefs" "${INTERSHEET_REFS}"
+			(at 123.2564 72.3106 0)
+			(effects
+				(font
+					(size 1.27 1.27)
+				)
+				(justify right)
+				(hide yes)
+			)
+		)
+	)
+	(global_label "ENABLE_SERVO_POWER_1"
+		(shape input)
+		(at 69.85 176.53 180)
+		(fields_autoplaced yes)
+		(effects
+			(font
+				(size 1.27 1.27)
+			)
+			(justify right)
+		)
+		(property "Intersheetrefs" "${INTERSHEET_REFS}"
+			(at 43.2188 176.53 0)
+			(effects
+				(font
+					(size 1.27 1.27)
+				)
+				(justify right)
+				(hide yes)
+			)
+		)
+	)
+	(global_label "SERVO_6"
+		(shape input)
+		(at 201.93 124.46 180)
+		(fields_autoplaced yes)
+		(effects
+			(font
+				(size 1.27 1.27)
+			)
+			(justify right)
+		)
+		(property "Intersheetrefs" "${INTERSHEET_REFS}"
+			(at 191.2921 124.3806 0)
+			(effects
+				(font
+					(size 1.27 1.27)
+				)
+				(justify right)
+				(hide yes)
+			)
 		)
 	)
 	(global_label "SERVO_8"
 		(shape input)
+		(at 201.93 147.32 180)
+		(fields_autoplaced yes)
+		(effects
+			(font
+				(size 1.27 1.27)
+			)
+			(justify right)
+		)
+		(property "Intersheetrefs" "${INTERSHEET_REFS}"
+			(at 191.2921 147.2406 0)
+			(effects
+				(font
+					(size 1.27 1.27)
+				)
+				(justify right)
+				(hide yes)
+			)
+		)
+	)
+	(global_label "SERVO_5"
+		(shape input)
 		(at 201.93 109.22 180)
 		(fields_autoplaced yes)
@@
 	(global_label "GND"
 		(shape input)
-		(at 129.54 72.39 180)
-		(fields_autoplaced yes)
-		(effects
-			(font
-				(size 1.27 1.27)
-			)
-			(justify right)
-		)
-		(property "Intersheetrefs" "${INTERSHEET_REFS}"
-			(at 123.2564 72.3106 0)
-			(effects
-				(font
-					(size 1.27 1.27)
-				)
-				(justify right)
-				(hide yes)
-			)
-		)
-	)
-	(global_label "ENABLE_SERVO_POWER_1"
-		(shape input)
-		(at 69.85 176.53 180)
-		(fields_autoplaced yes)
-		(effects
-			(font
-				(size 1.27 1.27)
-			)
-			(justify right)
-		)
-		(property "Intersheetrefs" "${INTERSHEET_REFS}"
-			(at 43.2188 176.53 0)
-			(effects
-				(font
-					(size 1.27 1.27)
-				)
-				(justify right)
-				(hide yes)
-			)
-		)
-	)
-	(global_label "SERVO_6"
-		(shape input)
-		(at 201.93 147.32 180)
-		(fields_autoplaced yes)
-		(effects
-			(font
-				(size 1.27 1.27)
-			)
-			(justify right)
-		)
-		(property "Intersheetrefs" "${INTERSHEET_REFS}"
-			(at 191.2921 147.2406 0)
-			(effects
-				(font
-					(size 1.27 1.27)
-				)
-				(justify right)
-				(hide yes)
-			)
-		)
-	)
-	(global_label "GND"
-		(shape input)
 		(at 129.54 81.28 180)
 		(fields_autoplaced yes)
@@
 		)
 	)
-	(global_label "SERVO_7"
+	(global_label "SERVO_2"
+		(shape input)
+		(at 201.93 68.58 180)
+		(fields_autoplaced yes)
+		(effects
+			(font
+				(size 1.27 1.27)
+			)
+			(justify right)
+		)
+		(property "Intersheetrefs" "${INTERSHEET_REFS}"
+			(at 191.2921 68.5006 0)
+			(effects
+				(font
+					(size 1.27 1.27)
+				)
+				(justify right)
+				(hide yes)
+			)
+		)
+	)
+	(global_label "SERVO_1"
+		(shape input)
+		(at 201.93 57.15 180)
+		(fields_autoplaced yes)
+		(effects
+			(font
+				(size 1.27 1.27)
+			)
+			(justify right)
+		)
+		(property "Intersheetrefs" "${INTERSHEET_REFS}"
+			(at 191.2921 57.0706 0)
+			(effects
+				(font
+					(size 1.27 1.27)
+				)
+				(justify right)
+				(hide yes)
+			)
+		)
+	)
+	(global_label "SERVO_3"
+		(shape input)
+		(at 201.93 80.01 180)
+		(fields_autoplaced yes)
+		(effects
+			(font
+				(size 1.27 1.27)
+			)
+			(justify right)
+		)
+		(property "Intersheetrefs" "${INTERSHEET_REFS}"
+			(at 191.2921 79.9306 0)
+			(effects
+				(font
+					(size 1.27 1.27)
+				)
+				(justify right)
+				(hide yes)
+			)
+		)
+	)
+	(global_label "SERVO_4"
 		(shape input)
 		(at 201.93 93.98 180)
@@
 			(effects
 				(font
-					(size 1.27 1.27)
-				)
-				(justify right)
-				(hide yes)
-			)
-		)
-	)
-	(global_label "SERVO_4"
-		(shape input)
-		(at 201.93 124.46 180)
-		(fields_autoplaced yes)
-		(effects
-			(font
-				(size 1.27 1.27)
-			)
-			(justify right)
-		)
-		(property "Intersheetrefs" "${INTERSHEET_REFS}"
-			(at 191.2921 124.3806 0)
-			(effects
-				(font
-					(size 1.27 1.27)
-				)
-				(justify right)
-				(hide yes)
-			)
-		)
-	)
-	(global_label "SERVO_2"
-		(shape input)
-		(at 201.93 68.58 180)
-		(fields_autoplaced yes)
-		(effects
-			(font
-				(size 1.27 1.27)
-			)
-			(justify right)
-		)
-		(property "Intersheetrefs" "${INTERSHEET_REFS}"
-			(at 191.2921 68.5006 0)
-			(effects
-				(font
-					(size 1.27 1.27)
-				)
-				(justify right)
-				(hide yes)
-			)
-		)
-	)
-	(global_label "SERVO_5"
-		(shape input)
-		(at 201.93 135.89 180)
-		(fields_autoplaced yes)
-		(effects
-			(font
-				(size 1.27 1.27)
-			)
-			(justify right)
-		)
-		(property "Intersheetrefs" "${INTERSHEET_REFS}"
-			(at 191.2921 135.8106 0)
-			(effects
-				(font
-					(size 1.27 1.27)
-				)
-				(justify right)
-				(hide yes)
-			)
-		)
-	)
-	(global_label "SERVO_1"
-		(shape input)
-		(at 201.93 57.15 180)
-		(fields_autoplaced yes)
-		(effects
-			(font
-				(size 1.27 1.27)
-			)
-			(justify right)
-		)
-		(property "Intersheetrefs" "${INTERSHEET_REFS}"
-			(at 191.2921 57.0706 0)
-			(effects
-				(font
-					(size 1.27 1.27)
-				)
-				(justify right)
-				(hide yes)
-			)
-		)
-	)
-	(global_label "SERVO_3"
-		(shape input)
-		(at 201.93 80.01 180)
-		(fields_autoplaced yes)
-		(effects
-			(font
-				(size 1.27 1.27)
-			)
-			(justify right)
-		)
-		(property "Intersheetrefs" "${INTERSHEET_REFS}"
-			(at 191.2921 79.9306 0)
-			(effects
-				(font
