File: servo_DCDC.kicad_sch (KiCad schematic)
At the start: 16 parts, among them Q7 CSD17307Q5A, Q8 CSD17579Q5A, U9 LM3150MH

Commit message: 12V logic for ESP32 + add legends + fine tune
Parts:
- added C30: 47uF, Capacitor_SMD:C_1210_3225Metric, symbol Device:C_Polarized
Connections:
- net GND: now also C30.2
- net VOUT: now also C30.1
Changed lines of the file:
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@@
+	)
+	(junction
+		(at 226.06 82.55)
+		(diameter 0)
+		(color 0 0 0 0)
 	)
 	(junction
@@
 	)
 	(junction
+		(at 214.63 93.98)
+		(diameter 0)
+		(color 0 0 0 0)
+	)
+	(junction
 		(at 161.29 93.98)
 		(diameter 0)
@@
 	(wire
 		(pts
-			(xy 214.63 82.55) (xy 227.33 82.55)
+			(xy 214.63 82.55) (xy 226.06 82.55)
 		)
 		(stroke
@@
 	(wire
 		(pts
+			(xy 226.06 93.98) (xy 214.63 93.98)
+		)
+		(stroke
+			(width 0)
+			(type default)
+		)
+	)
+	(wire
+		(pts
 			(xy 196.85 90.17) (xy 196.85 93.98)
 		)
@@
 	(wire
 		(pts
+			(xy 226.06 90.17) (xy 226.06 93.98)
+		)
+		(stroke
+			(width 0)
+			(type default)
+		)
+	)
+	(wire
+		(pts
 			(xy 173.99 93.98) (xy 161.29 93.98)
 		)
@@
 		(pts
 			(xy 119.38 83.82) (xy 130.81 83.82)
+		)
+		(stroke
+			(width 0)
+			(type default)
+		)
+	)
+	(wire
+		(pts
+			(xy 226.06 82.55) (xy 227.33 82.55)
 		)
 		(stroke
@@
 					(unit 1)
 				)
+			)
+		)
+	)
+	(symbol
+		(lib_id "Device:C_Polarized")
+		(at 226.06 86.36 0)
+		(unit 1)
+		(exclude_from_sim no)
+		(in_bom yes)
+		(on_board yes)
+		(dnp no)
+		(fields_autoplaced yes)
+		(property "Reference" "C30"
+			(at 229.87 84.2009 0)
+			(effects
+				(font
+					(size 1.27 1.27)
+				)
+				(justify left)
+			)
+		)
+		(property "Value" "47uF"
+			(at 229.87 86.7409 0)
+			(effects
+				(font
+					(size 1.27 1.27)
+				)
+				(justify left)
+			)
+		)
+		(property "Footprint" "Capacitor_SMD:C_1210_3225Metric"
+			(at 227.0252 90.17 0)
+			(effects
+				(font
+					(size 1.27 1.27)
+				)
+				(hide yes)
+			)
+		)
+		(property "Datasheet" "~"
+			(at 226.06 86.36 0)
+			(effects
+				(font
+					(size 1.27 1.27)
+				)
+				(hide yes)
+			)
+		)
+		(property "Description" "Polarized capacitor"
+			(at 226.06 86.36 0)
+			(effects
+				(font
+					(size 1.27 1.27)
+				)
+				(hide yes)
+			)
+		)
+		(pin "2"
+		)
+		(pin "1"
+		)
+		(instances
+			(project "carte_servo"
+				(path "/e63e39d7-6ac0-4ffd-8aa3-1841a4541b55/b1050287-31e3-44fe-9bba-b0376ddc40c3"
+					(reference "C30")
+					(unit 1)
+				)
