File: servo_DCDC.kicad_sch (KiCad schematic)
At the start: 17 parts, among them Q7 CSD17307Q5A, Q8 CSD17579Q5A, U9 LM3150MH

Commit message: Add BOM
Add LCSC reference and correct few footprint acording bom
Parts:
- C13: LCSC# (none) -> C19110
- C14: LCSC# (none) -> C7503496
- C15: LCSC# (none) -> C62782
- C16, C17, C30: LCSC# (none) -> C5440143
- C18: LCSC# (none) -> C57112
- C19, C20: LCSC# (none) -> C1713
- L1: Availability In Stock -> (none); Check_prices https://www.snapeda.com/parts/XAL6030-122MEC/Coilcraft/view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 -> (none); Description_1 1.2 µH Shielded Molded Inductor 16 A 7.5mOhm Max Nonstandard -> (none); LCSC# (none) -> C19191689; MANUFACTURER Coilcraft -> (none); MAXIMUM_PACKAGE_HEIGHT 3.1mm -> (none); MF Coilcraft -> (none); MP XAL6030-122MEC -> (none); PARTREV 11/02/18 -> (none); Package None -> (none); Price None -> (none); STANDARD Manufacturer Recommendations -> (none); SnapEDA_Link https://www.snapeda.com/parts/XAL6030-122MEC/Coilcraft/view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 -> (none)
- Q7: LCSC# (none) -> C22367097
- Q8: LCSC# (none) -> C2760461
- R1: LCSC# (none) -> C2930053
- R31: value 52.3k -> 52.3kR; footprint Capacitor_SMD:C_0603_1608Metric -> Resistor_SMD:R_0603_1608Metric; LCSC# (none) -> C23198
- R32: LCSC# (none) -> C2999456
- R33: LCSC# (none) -> C2933269
- U9: LCSC# (none) -> C1519420
Changed lines of the file:
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@@
 	(label "SW"
 		(at 124.46 78.74 0)
-		(fields_autoplaced yes)
 		(effects
 			(font
@@
 		(shape input)
 		(at 173.99 105.41 0)
-		(fields_autoplaced yes)
 		(effects
 			(font
@@
 		(shape input)
 		(at 97.79 104.14 0)
-		(fields_autoplaced yes)
 		(effects
 			(font
@@
 		(shape input)
 		(at 64.77 96.52 0)
-		(fields_autoplaced yes)
 		(effects
 			(font
@@
 		(shape input)
 		(at 54.61 69.85 0)
-		(fields_autoplaced yes)
 		(effects
 			(font
@@
 		(shape passive)
 		(at 81.28 99.06 0)
-		(fields_autoplaced yes)
 		(effects
 			(font
@@
 		(shape input)
 		(at 43.18 57.15 180)
-		(fields_autoplaced yes)
 		(effects
 			(font
@@
 		(shape input)
 		(at 205.74 99.06 0)
-		(fields_autoplaced yes)
 		(effects
 			(font
@@
 		(shape output)
 		(at 227.33 82.55 0)
-		(fields_autoplaced yes)
 		(effects
 			(font
@@
 		(shape input)
 		(at 130.81 105.41 0)
-		(fields_autoplaced yes)
 		(effects
 			(font
@@
 		(shape input)
 		(at 80.01 71.12 180)
-		(fields_autoplaced yes)
 		(effects
 			(font
@@
 			)
 		)
+		(property "LCSC#" "C2999456"
+			(at 173.99 86.36 0)
+			(effects
+				(font
+					(size 1.27 1.27)
+				)
+				(hide yes)
+			)
+		)
 		(pin "2"
 		)
@@
 			)
 		)
+		(property "LCSC#" "C5440143"
+			(at 214.63 86.36 0)
+			(effects
+				(font
+					(size 1.27 1.27)
+				)
+				(hide yes)
+			)
+		)
 		(pin "2"
 		)
@@
 			)
 		)
+		(property "LCSC#" "C2933269"
+			(at 173.99 100.33 0)
+			(effects
+				(font
+					(size 1.27 1.27)
+				)
+				(hide yes)
+			)
+		)
 		(pin "2"
 		)
@@
 			)
 		)
-		(property "Value" "52.3k"
+		(property "Value" "52.3kR"
 			(at 71.12 78.7399 0)
 			(effects
@@
 			)
 		)
-		(property "Footprint" "Capacitor_SMD:C_0603_1608Metric"
+		(property "Footprint" "Resistor_SMD:R_0603_1608Metric"
 			(at 68.58 77.47 0)
 			(effects
@@
 			)
 		)
+		(property "LCSC#" "C23198"
+			(at 68.58 77.47 0)
+			(effects
+				(font
+					(size 1.27 1.27)
+				)
+				(hide yes)
+			)
+		)
 		(pin "2"
 		)
@@
 			)
 		)
+		(property "LCSC#" "C1519420"
+			(at 97.79 81.28 0)
+			(effects
+				(font
+					(size 1.27 1.27)
+				)
+				(hide yes)
+			)
+		)
 		(pin "11"
 		)
@@
 			)
 		)
+		(property "LCSC#" "C1713"
+			(at 58.42 60.96 0)
+			(effects
+				(font
+					(size 1.27 1.27)
+				)
+				(hide yes)
+			)
+		)
 		(pin "2"
 		)
@@
 			)
 		)
+		(property "LCSC#" "C19110"
+			(at 64.77 90.17 0)
+			(effects
+				(font
+					(size 1.27 1.27)
+				)
+				(hide yes)
+			)
+		)
 		(pin "2"
 		)
@@
 			)
 		)
-		(property "MF" "Coilcraft"
+		(property "LCSC#" "C19191689"
 			(at 144.78 82.55 0)
 			(effects
@@
 					(size 1.27 1.27)
 				)
-				(justify bottom)
-				(hide yes)
-			)
-		)
-		(property "MAXIMUM_PACKAGE_HEIGHT" "3.1mm"
-			(at 144.78 82.55 0)
-			(effects
-				(font
-					(size 1.27 1.27)
-				)
-				(justify bottom)
-				(hide yes)
-			)
-		)
-		(property "Package" "None"
-			(at 144.78 82.55 0)
-			(effects
-				(font
-					(size 1.27 1.27)
-				)
-				(justify bottom)
-				(hide yes)
-			)
-		)
-		(property "Price" "None"
-			(at 144.78 82.55 0)
-			(effects
-				(font
-					(size 1.27 1.27)
-				)
-				(justify bottom)
-				(hide yes)
-			)
-		)
-		(property "Check_prices" "https://www.snapeda.com/parts/XAL6030-122MEC/Coilcraft/view-part/?ref=eda"
-			(at 144.78 82.55 0)
-			(effects
-				(font
-					(size 1.27 1.27)
-				)
-				(justify bottom)
-				(hide yes)
-			)
-		)
-		(property "STANDARD" "Manufacturer Recommendations"
-			(at 144.78 82.55 0)
-			(effects
-				(font
-					(size 1.27 1.27)
-				)
-				(justify bottom)
-				(hide yes)
-			)
-		)
-		(property "PARTREV" "11/02/18"
-			(at 144.78 82.55 0)
-			(effects
-				(font
-					(size 1.27 1.27)
-				)
-				(justify bottom)
-				(hide yes)
-			)
-		)
-		(property "SnapEDA_Link" "https://www.snapeda.com/parts/XAL6030-122MEC/Coilcraft/view-part/?ref=snap"
-			(at 144.78 82.55 0)
-			(effects
-				(font
-					(size 1.27 1.27)
-				)
-				(justify bottom)
-				(hide yes)
-			)
-		)
-		(property "MP" "XAL6030-122MEC"
-			(at 144.78 82.55 0)
-			(effects
-				(font
-					(size 1.27 1.27)
-				)
-				(justify bottom)
-				(hide yes)
-			)
-		)
-		(property "Description_1" "\n                        \n                            1.2 µH Shielded Molded Inductor 16 A 7.5mOhm Max Nonstandard\n                        \n"
-			(at 144.78 82.55 0)
-			(effects
-				(font
-					(size 1.27 1.27)
-				)
-				(justify bottom)
-				(hide yes)
-			)
-		)
-		(property "Availability" "In Stock"
-			(at 144.78 82.55 0)
-			(effects
-				(font
-					(size 1.27 1.27)
-				)
-				(justify bottom)
-				(hide yes)
-			)
-		)
-		(property "MANUFACTURER" "Coilcraft"
-			(at 144.78 82.55 0)
-			(effects
-				(font
-					(size 1.27 1.27)
-				)
-				(justify bottom)
 				(hide yes)
 			)
@@
 			)
 		)
+		(property "LCSC#" "C2930053"
+			(at 116.84 83.82 0)
+			(effects
+				(font
+					(size 1.27 1.27)
+				)
+				(hide yes)
+			)
+		)
 		(pin "2"
 		)
@@
 			)
 		)
+		(property "LCSC#" "C57112"
+			(at 81.28 92.71 0)
+			(effects
+				(font
+					(size 1.27 1.27)
+				)
+				(hide yes)
+			)
+		)
 		(pin "2"
 		)
@@
 			)
 		)
+		(property "LCSC#" "C5440143"
+			(at 196.85 86.36 0)
+			(effects
+				(font
+					(size 1.27 1.27)
+				)
+				(hide yes)
+			)
+		)
 		(pin "2"
 		)
@@
 			)
 		)
+		(property "LCSC#" "C2760461"
+			(at 128.27 100.33 0)
+			(effects
+				(font
+					(size 1.27 1.27)
+				)
+				(hide yes)
+			)
+		)
 		(pin "1"
 		)
@@
 			)
 		)
+		(property "LCSC#" "C5440143"
+			(at 226.06 86.36 0)
+			(effects
+				(font
+					(size 1.27 1.27)
+				)
+				(hide yes)
+			)
+		)
 		(pin "2"
 		)
@@
 			)
 		)
+		(property "LCSC#" "C1713"
+			(at 49.53 60.96 0)
+			(effects
+				(font
+					(size 1.27 1.27)
+				)
+				(hide yes)
+			)
+		)
 		(pin "2"
 		)
@@
 			)
 		)
+		(property "LCSC#" "C7503496"
+			(at 118.11 73.66 0)
+			(effects
+				(font
+					(size 1.27 1.27)
+				)
+				(hide yes)
+			)
+		)
 		(pin "2"
 		)
@@
 			)
 		)
+		(property "LCSC#" "C62782"
+			(at 161.29 86.36 0)
+			(effects
+				(font
+					(size 1.27 1.27)
+				)
+				(hide yes)
+			)
+		)
 		(pin "2"
 		)
@@
 			(at 128.27 71.12 0)
 			(effects
+				(font
+					(size 1.27 1.27)
+				)
+				(hide yes)
+			)
+		)
+		(property "LCSC#" "C22367097"
+			(at 128.27 71.12 0)
+			(effects

Commit message: prepare DCDC 24V compatibility + add reset/boot connector
Parts:
- C18: value 10nF -> 10nF (12V) - 15nF (24V)
- R31: value 52.3kR -> 52.3kR (12V) - 42.2kR (24V)
Other:
- note added: "24V input: XAL6030-182MEB (même empreinte) CSD18504Q5A (même empreinte) CSD18563Q5A (même empreinte)"
Changed lines of the file:
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@@
+		)
+	)
+	(text "24V input:\n	\nXAL6030-182MEB (même empreinte)\n\n	\nCSD18504Q5A (même empreinte)\n	\nCSD18563Q5A (même empreinte)"
+		(exclude_from_sim no)
+		(at 192.786 38.1 0)
+		(effects
+			(font
+				(size 1.27 1.27)
+			)
 		)
 	)
@@
 		(on_board yes)
 		(dnp no)
-		(fields_autoplaced yes)
 		(property "Reference" "R31"
 			(at 71.12 76.1999 0)
@@
 			)
 		)
-		(property "Value" "52.3kR"
-			(at 71.12 78.7399 0)
+		(property "Value" "52.3kR (12V) - 42.2kR (24V)"
+			(at 36.576 77.724 0)
 			(effects
 				(font
@@
 		(on_board yes)
 		(dnp no)
-		(fields_autoplaced yes)
 		(property "Reference" "C18"
 			(at 85.09 91.4399 0)
@@
 			)
 		)
-		(property "Value" "10nF"
-			(at 85.09 93.9799 0)
-			(effects
-				(font
+		(property "Value" "10nF (12V) - 15nF (24V)"
+			(at 68.58 102.616 0)
+			(effects
+				(font

Commit message: update to Kicad 9 + small fixes
Parts:
- U9: footprint Package_SO:HTSSOP-14-1EP_4.4x5mm_P0.65mm_EP3.4x5mm_Mask3x3.1mm -> Package_SO:Texas_HTSSOP-14-1EP_4.4x5mm_P0.65mm_EP3.4x5mm_Mask3.155x3.255mm

Commit message: update BOM
Parts:
- R1: value 1.74k -> 1.74kR
- R32: value 88.7k -> 88.7kR
- R33: value 9.76k -> 9.76kR
Changed lines of the file:
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@@
 			)
 		)
-		(property "Value" "88.7k"
+		(property "Value" "88.7kR"
 			(at 176.53 87.6299 0)
 			(effects
@@
 			)
 		)
-		(property "Value" "9.76k"
+		(property "Value" "9.76kR"
 			(at 176.53 101.5999 0)
 			(effects
@@
 			)
 		)
-		(property "Value" "1.74k"
+		(property "Value" "1.74kR"
 			(at 116.84 81.28 90)
 			(effects

Commit message: update BOM + add big capas (do not take DNP into account)
Parts:
- C13, C14, C15, R1, R32, R33: now not fitted
- C18: LCSC# C57112 -> C296713
- C19, C20: LCSC# C1713 -> C440198
- L1: value XAL6030-122MEC -> XAL6030-182MEB; LCSC# C19191689 -> C19191693
- Q7: LCSC# C22367097 -> C78118
- R31: LCSC# C23198 -> C23167
Other:
- note added: "12V input: L2 XAL6030-122MEC C19191689 (même empreinte) haut CSD17307Q5A C22367097 (même empreinte) bas CSD17579Q5A CSD17579Q5A (même empreinte)"
- note added: "24V input: L2 XAL6030-182MEB C19191693 (même empreinte) haut CSD18504Q5A C78118 (même empreinte) bas CSD18563Q5A C2760461 (même empreinte)"
- note removed: "24V input: XAL6030-182MEB (même empreinte) CSD18504Q5A (même empreinte) CSD18563Q5A (même empreinte)"
Changed lines of the file:
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@@
 	(generator_version "9.0")
 	(paper "A4")
-	(text "24V input:\n	\nXAL6030-182MEB (même empreinte)\n\n	\nCSD18504Q5A (même empreinte)\n	\nCSD18563Q5A (même empreinte)"
+	(text "24V input:\n	\nL2 XAL6030-182MEB C19191693 (même empreinte)\n\n	\nhaut CSD18504Q5A C78118 (même empreinte)\n	\nbas CSD18563Q5A C2760461 (même empreinte)"
 		(exclude_from_sim no)
 		(at 192.786 38.1 0)
+		(effects
+			(font
+				(size 1.27 1.27)
+			)
+		)
+	)
+	(text "12V input:\n	\nL2 XAL6030-122MEC C19191689 (même empreinte)\n\n	\nhaut CSD17307Q5A C22367097 (même empreinte)\n	\nbas CSD17579Q5A CSD17579Q5A (même empreinte)"
+		(exclude_from_sim no)
+		(at 140.97 37.846 0)
 		(effects
 			(font
@@
 		(in_bom yes)
 		(on_board yes)
-		(dnp no)
+		(dnp yes)
 		(fields_autoplaced yes)
 		(property "Reference" "R32"
@@
 		(in_bom yes)
 		(on_board yes)
-		(dnp no)
+		(dnp yes)
 		(fields_autoplaced yes)
 		(property "Reference" "R33"
@@
 			)
 		)
-		(property "LCSC#" "C23198"
+		(property "LCSC#" "C23167"
 			(at 68.58 77.47 0)
 			(effects
@@
 			)
 		)
-		(property "LCSC#" "C1713"
+		(property "LCSC#" "C440198"
 			(at 58.42 60.96 0)
 			(effects
@@
 		(in_bom yes)
 		(on_board yes)
-		(dnp no)
+		(dnp yes)
 		(fields_autoplaced yes)
 		(property "Reference" "C13"
@@
 			)
 		)
-		(property "Value" "XAL6030-122MEC"
+		(property "Value" "XAL6030-182MEB"
 			(at 144.78 78.74 0)
 			(effects
@@
 			)
 		)
-		(property "LCSC#" "C19191689"
+		(property "LCSC#" "C19191693"
 			(at 144.78 82.55 0)
 			(effects
@@
 		(in_bom yes)
 		(on_board yes)
-		(dnp no)
+		(dnp yes)
 		(fields_autoplaced yes)
 		(property "Reference" "R1"
@@
 			)
 		)
-		(property "LCSC#" "C57112"
+		(property "LCSC#" "C296713"
 			(at 81.28 92.71 0)
 			(effects
@@
 			)
 		)
-		(property "LCSC#" "C1713"
+		(property "LCSC#" "C440198"
 			(at 49.53 60.96 0)
 			(effects
@@
 		(in_bom yes)
 		(on_board yes)
-		(dnp no)
+		(dnp yes)
 		(fields_autoplaced yes)
 		(property "Reference" "C14"
@@
 		(in_bom yes)
 		(on_board yes)
-		(dnp no)
+		(dnp yes)
 		(fields_autoplaced yes)
 		(property "Reference" "C15"
@@
 			)
 		)
-		(property "LCSC#" "C22367097"
+		(property "LCSC#" "C78118"
 			(at 128.27 71.12 0)
 			(effects

Commit message: fix DNP (was just for checking what was to be bought)
Parts:
- C13, C14, C15, R1, R32, R33: now fitted
Changed lines of the file:
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@@
 		(in_bom yes)
 		(on_board yes)
-		(dnp yes)
+		(dnp no)
 		(fields_autoplaced yes)
 		(property "Reference" "R32"
@@
 		(in_bom yes)
 		(on_board yes)
-		(dnp yes)
+		(dnp no)
 		(fields_autoplaced yes)
 		(property "Reference" "R33"
@@
 		(in_bom yes)
 		(on_board yes)
-		(dnp yes)
+		(dnp no)
 		(fields_autoplaced yes)
 		(property "Reference" "C13"
@@
 		(in_bom yes)
 		(on_board yes)
-		(dnp yes)
+		(dnp no)
 		(fields_autoplaced yes)
 		(property "Reference" "R1"
@@
 		(in_bom yes)
 		(on_board yes)
-		(dnp yes)
+		(dnp no)
 		(fields_autoplaced yes)
 		(property "Reference" "C14"
@@
 		(in_bom yes)
 		(on_board yes)
-		(dnp yes)
+		(dnp no)
 		(fields_autoplaced yes)
 		(property "Reference" "C15"

Commit message: change capacitor references to support >25V
Parts:
- C14: LCSC# C7503496 -> C2905413
Changed lines of the file:
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@@
 			)
 		)
-		(property "LCSC#" "C7503496"
+		(property "LCSC#" "C2905413"
 			(at 118.11 73.66 0)
 			(effects
