File: carte_servo.kicad_sch (KiCad schematic)
At the start: 72 parts, among them J15 Conn_01x04_Pin, J16 Conn_01x05, J17 Conn_01x05, J2 Conn_02x04_Top_Bottom, J22 Conn_02x04_Top_Bottom, J23 Conn_01x05, J24 Conn_LEDs, SW1 SW_Reset, SW2 SW_Boot, U1 XGZP6897D_differential_pressu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

Commit message: fix warnings + add big capa on 6V DCDC input
Parts:
- added C43: C_Polarized, Capacitor_THT:CP_Radial_D7.5mm_P2.50mm, symbol Device:C_Polarized
Connections:
- net GND: now also C43.2
- net ServoDCDC/VIN: now also C43.1
Other:
- moved on the sheet: C29
Changed lines of the file:
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@@
 	(rectangle
 		(start 53.34 331.47)
-		(end 232.41 383.54)
+		(end 172.72 383.54)
 		(stroke
 			(width 0)
@@
 	(text "Voltmeters and enables"
 		(exclude_from_sim no)
-		(at 152.654 379.222 0)
+		(at 112.776 378.714 0)
 		(effects
 			(font
@@
 	)
 	(junction
-		(at 204.47 200.66)
+		(at 367.03 354.33)
 		(diameter 0)
 		(color 0 0 0 0)
 	)
 	(junction
-		(at 367.03 354.33)
+		(at 306.07 208.28)
 		(diameter 0)
 		(color 0 0 0 0)
 	)
 	(junction
-		(at 306.07 208.28)
+		(at 204.47 201.93)
 		(diameter 0)
 		(color 0 0 0 0)
@@
 	)
 	(junction
+		(at 444.5 54.61)
+		(diameter 0)
+		(color 0 0 0 0)
+	)
+	(junction
 		(at 398.78 308.61)
 		(diameter 0)
@@
 	)
 	(junction
+		(at 309.88 74.93)
+		(diameter 0)
+		(color 0 0 0 0)
+	)
+	(junction
 		(at 401.32 328.93)
 		(diameter 0)
@@
 	)
 	(junction
+		(at 213.36 201.93)
+		(diameter 0)
+		(color 0 0 0 0)
+	)
+	(junction
 		(at 302.26 330.2)
 		(diameter 0)
@@
 	(wire
 		(pts
+			(xy 213.36 201.93) (xy 204.47 201.93)
+		)
+		(stroke
+			(width 0)
+			(type default)
+		)
+	)
+	(wire
+		(pts
 			(xy 401.32 328.93) (xy 412.75 328.93)
 		)
@@
 	(wire
 		(pts
+			(xy 447.04 74.93) (xy 447.04 76.2)
+		)
+		(stroke
+			(width 0)
+			(type default)
+		)
+	)
+	(wire
+		(pts
 			(xy 473.71 186.69) (xy 478.79 186.69)
 		)
@@
 	(wire
 		(pts
+			(xy 309.88 74.93) (xy 311.15 74.93)
+		)
+		(stroke
+			(width 0)
+			(type default)
+		)
+	)
+	(wire
+		(pts
 			(xy 308.61 234.95) (xy 311.15 234.95)
 		)
@@
 	(wire
 		(pts
+			(xy 193.04 201.93) (xy 193.04 200.66)
+		)
+		(stroke
+			(width 0)
+			(type default)
+		)
+	)
+	(wire
+		(pts
 			(xy 144.78 52.07) (xy 140.97 52.07)
 		)
@@
 	(wire
 		(pts
-			(xy 204.47 200.66) (xy 213.36 200.66)
-		)
-		(stroke
-			(width 0)
-			(type default)
-		)
-	)
-	(wire
-		(pts
 			(xy 238.76 49.53) (xy 236.22 49.53)
 		)
@@
 	(wire
 		(pts
-			(xy 311.15 83.82) (xy 311.15 82.55)
-		)
-		(stroke
-			(width 0)
-			(type default)
-		)
-	)
-	(wire
-		(pts
 			(xy 74.93 179.07) (xy 74.93 176.53)
 		)
@@
 	(wire
 		(pts
-			(xy 435.61 54.61) (xy 448.31 54.61)
+			(xy 435.61 54.61) (xy 444.5 54.61)
 		)
 		(stroke
@@
 	(wire
 		(pts
-			(xy 204.47 200.66) (xy 204.47 203.2)
+			(xy 204.47 200.66) (xy 204.47 201.93)
 		)
 		(stroke
@@
 	(wire
 		(pts
+			(xy 447.04 76.2) (xy 444.5 76.2)
+		)
+		(stroke
+			(width 0)
+			(type default)
+		)
+	)
+	(wire
+		(pts
+			(xy 219.71 201.93) (xy 213.36 201.93)
+		)
+		(stroke
+			(width 0)
+			(type default)
+		)
+	)
+	(wire
+		(pts
 			(xy 302.26 327.66) (xy 304.8 327.66)
 		)
@@
 	(wire
 		(pts
-			(xy 308.61 74.93) (xy 311.15 74.93)
+			(xy 308.61 74.93) (xy 309.88 74.93)
 		)
 		(stroke
@@
 	(wire
 		(pts
+			(xy 444.5 54.61) (xy 448.31 54.61)
+		)
+		(stroke
+			(width 0)
+			(type default)
+		)
+	)
+	(wire
+		(pts
 			(xy 398.78 316.23) (xy 415.29 316.23)
 		)
@@
 	(wire
 		(pts
-			(xy 193.04 200.66) (xy 204.47 200.66)
+			(xy 193.04 201.93) (xy 204.47 201.93)
 		)
 		(stroke
@@
 	(wire
 		(pts
+			(xy 213.36 201.93) (xy 213.36 200.66)
+		)
+		(stroke
+			(width 0)
+			(type default)
+		)
+	)
+	(wire
+		(pts
 			(xy 63.5 187.96) (xy 63.5 184.15)
 		)
@@
 	(wire
 		(pts
+			(xy 311.15 76.2) (xy 311.15 74.93)
+		)
+		(stroke
+			(width 0)
+			(type default)
+		)
+	)
+	(wire
+		(pts
 			(xy 306.07 208.28) (xy 311.15 208.28)
 		)
@@
 	(wire
 		(pts
+			(xy 444.5 54.61) (xy 444.5 64.77)
+		)
+		(stroke
+			(width 0)
+			(type default)
+		)
+	)
+	(wire
+		(pts
 			(xy 177.8 77.47) (xy 194.31 77.47)
 		)
@@
 	(wire
 		(pts
-			(xy 311.15 72.39) (xy 311.15 74.93)
+			(xy 309.88 72.39) (xy 309.88 74.93)
 		)
 		(stroke
@@
 	(wire
 		(pts
-			(xy 302.26 72.39) (xy 311.15 72.39)
+			(xy 444.5 76.2) (xy 444.5 72.39)
+		)
+		(stroke
+			(width 0)
+			(type default)
+		)
+	)
+	(wire
+		(pts
+			(xy 302.26 72.39) (xy 309.88 72.39)
 		)
 		(stroke
@@
 	(global_label "GND"
 		(shape input)
-		(at 204.47 203.2 0)
+		(at 219.71 201.93 0)
 		(fields_autoplaced yes)
 		(effects
@@
 		)
 		(property "Intersheetrefs" "${INTERSHEET_REFS}"
-			(at 211.3257 203.2 0)
+			(at 226.5657 201.93 0)
 			(effects
 				(font
@@
 		)
 	)
+	(global_label "GND_POWER"
+		(shape output)
+		(at 447.04 74.93 0)
+		(fields_autoplaced yes)
+		(effects
+			(font
+				(size 1.27 1.27)
+			)
+			(justify left)
+		)
+		(property "Intersheetrefs" "${INTERSHEET_REFS}"
+			(at 461.3342 74.93 0)
+			(effects
+				(font
+					(size 1.27 1.27)
+				)
+				(justify left)
+				(hide yes)
+			)
+		)
+	)
 	(global_label "LEDs"
 		(shape output)
@@
 	)
 	(symbol
+		(lib_id "Device:C_Polarized")
+		(at 444.5 68.58 0)
+		(unit 1)
+		(exclude_from_sim no)
+		(in_bom yes)
+		(on_board yes)
+		(dnp no)
+		(property "Reference" "C43"
+			(at 436.626 68.072 0)
+			(effects
+				(font
+					(size 1.27 1.27)
+				)
+				(justify left)
+			)
+		)
+		(property "Value" "C_Polarized"
+			(at 430.022 70.612 0)
+			(effects
+				(font
+					(size 1.27 1.27)
+				)
+				(justify left)
+			)
+		)
+		(property "Footprint" "Capacitor_THT:CP_Radial_D7.5mm_P2.50mm"
+			(at 445.4652 72.39 0)
+			(effects
+				(font
+					(size 1.27 1.27)
+				)
+				(hide yes)
+			)
+		)
+		(property "Datasheet" "~"
+			(at 444.5 68.58 0)
+			(effects
+				(font
+					(size 1.27 1.27)
+				)
+				(hide yes)
+			)
+		)
+		(property "Description" "Polarized capacitor"
+			(at 444.5 68.58 0)
+			(effects
+				(font
+					(size 1.27 1.27)
+				)
+				(hide yes)
+			)
+		)
+		(property "LCSC#" "C398835"
+			(at 444.5 68.58 0)
+			(effects
+				(font
+					(size 1.27 1.27)
+				)
+				(hide yes)
+			)
+		)
+		(pin "1"
+		)
+		(pin "2"
+		)
+		(instances
+			(project "carte_servo"
+				(path "/e63e39d7-6ac0-4ffd-8aa3-1841a4541b55"
+					(reference "C43")
+					(unit 1)
+				)
+			)
+		)
+	)
+	(symbol
 		(lib_id "Device:Fuse")
 		(at 356.87 346.71 270)
@@
 	(symbol
 		(lib_id "Device:C")
-		(at 311.15 78.74 0)
+		(at 311.15 80.01 0)
 		(mirror y)
 		(unit 1)
@@
 		(dnp no)
 		(property "Reference" "C29"
-			(at 307.34 77.4699 0)
+			(at 307.34 78.7399 0)
 			(effects
 				(font
@@
 		)
 		(property "Value" "100nF"
-			(at 307.34 80.0099 0)
+			(at 307.34 81.2799 0)
 			(effects
 				(font
@@
 		)
 		(property "Footprint" "Capacitor_SMD:C_0603_1608Metric"
-			(at 310.1848 82.55 0)
+			(at 310.1848 83.82 0)
 			(effects
 				(font
@@
 		)
 		(property "Datasheet" "~"
-			(at 311.15 78.74 0)
+			(at 311.15 80.01 0)
 			(effects
 				(font
@@
 		)
 		(property "Description" "Unpolarized capacitor"
-			(at 311.15 78.74 0)
+			(at 311.15 80.01 0)
 			(effects
 				(font
@@
 		)
 		(property "LCSC#" "C14663"
-			(at 311.15 78.74 0)
+			(at 311.15 80.01 0)
 			(effects
 				(font
