File: USB_conn.kicad_sch (KiCad schematic)
At the start: 7 parts, among them P1 USB_C_Plug_USB2.0

Commit message: update to Kicad 9 + small fixes
Changed lines of the file:
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@@
 (kicad_sch
-	(version 20231120)
+	(version 20250114)
 	(generator "eeschema")
-	(generator_version "8.0")
+	(generator_version "9.0")
 	(paper "A4")
 	(junction
@@
 			)
 		)
+		(property "Sim.Device" "D"
+			(at 124.46 73.66 0)
+			(effects
+				(font
+					(size 1.27 1.27)
+				)
+				(hide yes)
+			)
+		)
+		(property "Sim.Pins" "1=K 2=A"
+			(at 124.46 73.66 0)
+			(effects
+				(font
+					(size 1.27 1.27)
+				)
+				(hide yes)
+			)
+		)
 		(pin "1"
 		)
@@
 			)
 		)
-		(property "Datasheet" "https://www.mouser.fr/ProductDetail/Texas-Instruments/ESD321DYAR?qs=rQFj71Wb1eXoYwRMra0IYA%3D%3D"
+		(property "Datasheet" "~"
 			(at 133.35 100.33 0)
 			(effects
@@
 			)
 		)
-		(property "Datasheet" "https://www.lcsc.com/product-detail/USB-Connectors_G-Switch-GT-USB-7047A_C963216.html"
+		(property "Datasheet" "https://www.usb.org/sites/default/files/documents/usb_type-c.zip"
 			(at 107.95 88.9 0)
 			(effects
@@
 			)
 		)
-		(property "Datasheet" "https://www.mouser.fr/ProductDetail/Texas-Instruments/ESD321DYAR?qs=rQFj71Wb1eXoYwRMra0IYA%3D%3D"
+		(property "Datasheet" "~"
 			(at 146.05 100.33 0)
 			(effects
