File: DCDC_5V.kicad_sch (KiCad schematic)
At the start: 12 parts, among them U10 TPS563200

Commit message: change capacitor references to support >25V
Parts:
- C24, C25: LCSC# C5674 -> C29277
Changed lines of the file:
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@@
 			)
 		)
-		(property "LCSC#" "C5674"
+		(property "LCSC#" "C29277"
 			(at 187.96 80.01 0)
 			(effects
@@
 			)
 		)
-		(property "LCSC#" "C5674"
+		(property "LCSC#" "C29277"
 			(at 198.12 80.01 0)
 			(effects
